File: 1sq_power_supply.sch (KiCad schematic (older format))
At the start: 46 parts, among them J1 TC2030-MCP, J2 Conn_01x02, J3 Conn_01x02, J4 Conn_01x02, J5 Conn_01x02, J6 Conn_01x05_Male, U1 L78L05_SOT89, U2 LM2596S-ADJ, U3 STM32F030F4Px, U4 AP2210N-3.3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

Commit message: added footprints
Parts:
- C10, C15, C16, C17, C3, C4, C5, C6, C7, C9: footprint (none) -> Capacitor_SMD:C_0603_1608Metric
- C11, C12, C13, C14, R1, R10, R11, R12, R13, R2, R3, R4, R5, R6, R7, R8, R9: footprint (none) -> Resistor_SMD:R_0603_1608Metric
- C2, C8: footprint (none) -> Capacitor_SMD:CP_Elec_8x10
- D1: footprint (none) -> Diode_SMD:D_SMB
- D2: footprint (none) -> Diode_SMD:D_SMA
- D3: footprint (none) -> Diode_SMD:D_0603_1608Metric
- J1: footprint Homebrew_TC2030-MCP -> Connector:Tag-Connect_TC2030-IDC-NL_2x03_P1.27mm_Vertical
- J2, J3, J4, J5: footprint (none) -> Connector_PinSocket_2.54mm:PinSocket_1x02_P2.54mm_Vertical
- J6: footprint (none) -> Connector_PinHeader_1.27mm:PinHeader_1x05_P1.27mm_Vertical
- L1: footprint (none) -> Inductor_SMD:L_12x12mm_H8mm
- OLEDM1: footprint (none) -> AdoptedTweaked:IROP055-SSD1306Z-PADS-ONLY
- R14: footprint (none) -> Resistor_SMD:R_2512_6332Metric
- U5: footprint (none) -> Package_SO:TSSOP-14_4.4x5mm_P0.65mm

Commit message: 2-22-19 update
Connections:
- wire segments 190 -> 192
Changed lines of the file:
@@
 L Device:C_Small C9
 U 1 1 5B7EC773
-P 6200 6600
-F 0 "C9" H 6292 6646 50  0000 L CNN
-F 1 "1u" H 6292 6555 50  0000 L CNN
-F 2 "Capacitor_SMD:C_0603_1608Metric" H 6200 6600 50  0001 C CNN
-F 3 "" H 6200 6600 50  0001 C CNN
-	1    6200 6600
+P 5500 4800
+F 0 "C9" H 5592 4846 50  0000 L CNN
+F 1 "1u" H 5592 4755 50  0000 L CNN
+F 2 "Capacitor_SMD:C_0603_1608Metric" H 5500 4800 50  0001 C CNN
+F 3 "" H 5500 4800 50  0001 C CNN
+	1    5500 4800
 	1    0    0    -1
 $EndComp
@@
 L Device:R_Small R9
 U 1 1 5B7EC8DA
-P 6000 6500
-F 0 "R9" V 5804 6500 50  0000 C CNN
-F 1 "1k5" V 5895 6500 50  0000 C CNN
-F 2 "Resistor_SMD:R_0603_1608Metric" H 6000 6500 50  0001 C CNN
-F 3 "" H 6000 6500 50  0001 C CNN
-	1    6000 6500
+P 5300 4700
+F 0 "R9" V 5104 4700 50  0000 C CNN
+F 1 "1k5" V 5195 4700 50  0000 C CNN
+F 2 "Resistor_SMD:R_0603_1608Metric" H 5300 4700 50  0001 C CNN
+F 3 "" H 5300 4700 50  0001 C CNN
+	1    5300 4700
 	0    1    1    0
 $EndComp
@@
 	1    0    0    -1
 $EndComp
+Text GLabel 5900 6400 0    50   Input ~ 0
+Vout
 Text GLabel 4900 6400 0    50   Input ~ 0
-Vout
-Text GLabel 4500 6600 0    50   Input ~ 0
 Vin
 $Comp
 L Device:R_Small R4
 U 1 1 5B81087A
-P 4500 6800
-F 0 "R4" H 4441 6754 50  0000 R CNN
-F 1 "R_Small" H 4441 6845 50  0000 R CNN
-F 2 "Resistor_SMD:R_0603_1608Metric" H 4500 6800 50  0001 C CNN
-F 3 "" H 4500 6800 50  0001 C CNN
-	1    4500 6800
+P 5000 6600
+F 0 "R4" H 4941 6554 50  0000 R CNN
+F 1 "R_Small" H 4941 6645 50  0000 R CNN
+F 2 "Resistor_SMD:R_0603_1608Metric" H 5000 6600 50  0001 C CNN
+F 3 "" H 5000 6600 50  0001 C CNN
+	1    5000 6600
 	-1   0    0    1
 $EndComp
@@
 L Device:R_Small R5
 U 1 1 5B8133E7
-P 4500 7200
-F 0 "R5" H 4441 7154 50  0000 R CNN
-F 1 "R_Small" H 4441 7245 50  0000 R CNN
-F 2 "Resistor_SMD:R_0603_1608Metric" H 4500 7200 50  0001 C CNN
-F 3 "" H 4500 7200 50  0001 C CNN
-	1    4500 7200
+P 5000 7100
+F 0 "R5" H 4941 7054 50  0000 R CNN
+F 1 "R_Small" H 4941 7145 50  0000 R CNN
+F 2 "Resistor_SMD:R_0603_1608Metric" H 5000 7100 50  0001 C CNN
+F 3 "" H 5000 7100 50  0001 C CNN
+	1    5000 7100
 	-1   0    0    1
 $EndComp
@@
 L Device:R_Small R6
 U 1 1 5B813433
-P 4900 6600
-F 0 "R6" H 4841 6554 50  0000 R CNN
-F 1 "R_Small" H 4841 6645 50  0000 R CNN
-F 2 "Resistor_SMD:R_0603_1608Metric" H 4900 6600 50  0001 C CNN
-F 3 "" H 4900 6600 50  0001 C CNN
-	1    4900 6600
+P 6000 6600
+F 0 "R6" H 5941 6554 50  0000 R CNN
+F 1 "R_Small" H 5941 6645 50  0000 R CNN
+F 2 "Resistor_SMD:R_0603_1608Metric" H 6000 6600 50  0001 C CNN
+F 3 "" H 6000 6600 50  0001 C CNN
+	1    6000 6600
 	-1   0    0    1
 $EndComp
@@
 L Device:R_Small R7
 U 1 1 5B813485
-P 4900 7100
-F 0 "R7" H 4841 7054 50  0000 R CNN
-F 1 "R_Small" H 4841 7145 50  0000 R CNN
-F 2 "Resistor_SMD:R_0603_1608Metric" H 4900 7100 50  0001 C CNN
-F 3 "" H 4900 7100 50  0001 C CNN
-	1    4900 7100
-	-1   0    0    1
-$EndComp
-$Comp
-L power:GND #PWR014
-U 1 1 5B813509
-P 4500 7300
-F 0 "#PWR014" H 4500 7050 50  0001 C CNN
-F 1 "GND" H 4505 7127 50  0000 C CNN
-F 2 "" H 4500 7300 50  0001 C CNN
-F 3 "" H 4500 7300 50  0001 C CNN
-	1    4500 7300
-	1    0    0    -1
-$EndComp
-$Comp
-L power:GND #PWR015
-U 1 1 5B81354A
-P 4900 7200
-F 0 "#PWR015" H 4900 6950 50  0001 C CNN
-F 1 "GND" H 4905 7027 50  0000 C CNN
-F 2 "" H 4900 7200 50  0001 C CNN
-F 3 "" H 4900 7200 50  0001 C CNN
-	1    4900 7200
-	1    0    0    -1
-$EndComp
-Text Label 4100 7000 0    50   ~ 0
-Vi_Sense
-Text Label 5300 6900 2    50   ~ 0
-Vo_Sense
-Wire Wire Line
-	4100 7000 4500 7000
-Wire Wire Line
-	4500 7000 4500 7100
-Wire Wire Line
-	4500 6900 4500 7000
-Connection ~ 4500 7000
-Wire Wire Line
-	4500 6600 4500 6700
-Wire Wire Line
-	4900 6400 4900 6500
-Wire Wire Line
-	4900 6700 4900 6900
-Wire Wire Line
-	5300 6900 4900 6900
-Connection ~ 4900 6900
-Wire Wire Line
-	4900 6900 4900 7000
-$Comp
-L Device:C_Small C10
-U 1 1 5B81C0DA
-P 6200 7200
-F 0 "C10" H 6292 7246 50  0000 L CNN
-F 1 "1u" H 6292 7155 50  0000 L CNN
-F 2 "Capacitor_SMD:C_0603_1608Metric" H 6200 7200 50  0001 C CNN
-F 3 "" H 6200 7200 50  0001 C CNN
-	1    6200 7200
-	1    0    0    -1
-$EndComp
-$Comp
-L Device:R_Small R10
-U 1 1 5B81C0E0
 P 6000 7100
-F 0 "R10" V 5804 7100 50  0000 C CNN
-F 1 "1k5" V 5895 7100 50  0000 C CNN
+F 0 "R7" H 5941 7054 50  0000 R CNN
+F 1 "R_Small" H 5941 7145 50  0000 R CNN
 F 2 "Resistor_SMD:R_0603_1608Metric" H 6000 7100 50  0001 C CNN
 F 3 "" H 6000 7100 50  0001 C CNN
 	1    6000 7100
+	-1   0    0    1
+$EndComp
+$Comp
+L power:GND #PWR014
+U 1 1 5B813509
+P 5000 7200
+F 0 "#PWR014" H 5000 6950 50  0001 C CNN
+F 1 "GND" H 5005 7027 50  0000 C CNN
+F 2 "" H 5000 7200 50  0001 C CNN
+F 3 "" H 5000 7200 50  0001 C CNN
+	1    5000 7200
+	1    0    0    -1
+$EndComp
+$Comp
+L power:GND #PWR015
+U 1 1 5B81354A
+P 6000 7200
+F 0 "#PWR015" H 6000 6950 50  0001 C CNN
+F 1 "GND" H 6005 7027 50  0000 C CNN
+F 2 "" H 6000 7200 50  0001 C CNN
+F 3 "" H 6000 7200 50  0001 C CNN
+	1    6000 7200
+	1    0    0    -1
+$EndComp
+Text Label 4600 6900 0    50   ~ 0
+Vi_Sense
+Text Label 6400 6900 2    50   ~ 0
+Vo_Sense
+Wire Wire Line
+	4600 6900 5000 6900
+Wire Wire Line
+	5000 6900 5000 7000
+Wire Wire Line
+	5000 6700 5000 6900
+Connection ~ 5000 6900
+Wire Wire Line
+	4900 6400 5000 6400
+Wire Wire Line
+	6000 6400 6000 6500
+Wire Wire Line
+	6000 6700 6000 6900
+Wire Wire Line
+	6400 6900 6000 6900
+Connection ~ 6000 6900
+Wire Wire Line
+	6000 6900 6000 7000
+$Comp
+L Device:C_Small C10
+U 1 1 5B81C0DA
+P 5500 5400
+F 0 "C10" H 5592 5446 50  0000 L CNN
+F 1 "1u" H 5592 5355 50  0000 L CNN
+F 2 "Capacitor_SMD:C_0603_1608Metric" H 5500 5400 50  0001 C CNN
+F 3 "" H 5500 5400 50  0001 C CNN
+	1    5500 5400
+	1    0    0    -1
+$EndComp
+$Comp
+L Device:R_Small R10
+U 1 1 5B81C0E0
+P 5300 5300
+F 0 "R10" V 5104 5300 50  0000 C CNN
+F 1 "1k5" V 5195 5300 50  0000 C CNN
+F 2 "Resistor_SMD:R_0603_1608Metric" H 5300 5300 50  0001 C CNN
+F 3 "" H 5300 5300 50  0001 C CNN
+	1    5300 5300
 	0    1    1    0
 $EndComp
@@
 L power:GND #PWR019
 U 1 1 5B81CCD3
-P 6200 7300
-F 0 "#PWR019" H 6200 7050 50  0001 C CNN
-F 1 "GND" H 6205 7127 50  0000 C CNN
-F 2 "" H 6200 7300 50  0001 C CNN
-F 3 "" H 6200 7300 50  0001 C CNN
-	1    6200 7300
+P 5500 5500
+F 0 "#PWR019" H 5500 5250 50  0001 C CNN
+F 1 "GND" H 5505 5327 50  0000 C CNN
+F 2 "" H 5500 5500 50  0001 C CNN
+F 3 "" H 5500 5500 50  0001 C CNN
+	1    5500 5500
 	1    0    0    -1
 $EndComp
@@
 L power:GND #PWR018
 U 1 1 5B81CD18
-P 6200 6700
-F 0 "#PWR018" H 6200 6450 50  0001 C CNN
-F 1 "GND" H 6205 6527 50  0000 C CNN
-F 2 "" H 6200 6700 50  0001 C CNN
-F 3 "" H 6200 6700 50  0001 C CNN
-	1    6200 6700
-	1    0    0    -1
-$EndComp
-Wire Wire Line
-	6100 6500 6200 6500
-Wire Wire Line
-	6200 6500 6500 6500
-Connection ~ 6200 6500
-Wire Wire Line
-	6500 7100 6200 7100
-Wire Wire Line
-	6200 7100 6100 7100
-Connection ~ 6200 7100
-Text Label 5500 6500 0    50   ~ 0
+P 5500 4900
+F 0 "#PWR018" H 5500 4650 50  0001 C CNN
+F 1 "GND" H 5505 4727 50  0000 C CNN
+F 2 "" H 5500 4900 50  0001 C CNN
+F 3 "" H 5500 4900 50  0001 C CNN
+	1    5500 4900
+	1    0    0    -1
+$EndComp
+Wire Wire Line
+	5400 4700 5500 4700
+Wire Wire Line
+	5500 4700 5800 4700
+Connection ~ 5500 4700
+Wire Wire Line
+	5800 5300 5500 5300
+Wire Wire Line
+	5500 5300 5400 5300
+Connection ~ 5500 5300
+Text Label 4800 4700 0    50   ~ 0
 V_Target
-Text Label 5500 7100 0    50   ~ 0
+Text Label 4800 5300 0    50   ~ 0
 A_Limit
 Wire Wire Line
-	5500 7100 5900 7100
-Wire Wire Line
-	5500 6500 5900 6500
-Text Label 6500 6500 2    50   ~ 0
+	4800 5300 5200 5300
+Wire Wire Line
+	4800 4700 5200 4700
+Text Label 5800 4700 2    50   ~ 0
 Vset
-Text Label 6500 7100 2    50   ~ 0
+Text Label 5800 5300 2    50   ~ 0
 Aset
 Text Label 5700 1500 0    50   ~ 0
@@
 Wire Wire Line
 	2400 6300 3000 6300
+Wire Wire Line
+	5000 6400 5000 6500
+Wire Wire Line
+	5900 6400 6000 6400
 $EndSCHEMATC
